File: hardware/mdx1/ui_audio_rf.kicad_sch (KiCad schematic)
At the start: 36 parts, among them J7 UI link FFC 20p 0.5mm, J8 3.5 mm jack, J9 Speaker 8R, Q8 2N7002, U23 LSM6DSM (IMU), U24 TPA6132A2 (HP amp), U25 PAM8302A (2.5 W class-D), U26 BM83SM1-00AA, U27 MAX-M10S (GNSS), U28 GNSS chip antenna

Commit message: Re-source out-of-stock parts; rework D8/9 footprint and GNSS antenna front end
Parts re-sourced to in-stock equivalents (BOM + board + firmware kept in sync):
- U4  TPS65131RGET, U12 INA241A2QDGKRQ1, U23 LSM6DSO32TR (same footprints)
- Q1  SiR680ADP-T1-UE3 (80 V, same PowerPAK SO-8; higher Qg - verify gate drive)
- U2  BQ27441DRZT-G1A (drop-in, R9 sense retained)
- D8/9 NSVBAT54SWT1G: SOT-323/SC-70 dual-series wired as a single diode
  (anode=pin1, cathode=pin3, pin2 NC); footprint changed on the board
- C32/C33/C38-48 re-sourced (KEMET/Murata/TDK), same footprints

GNSS antenna: chip antenna -> external active antenna via u.FL
- Removed U28 (chip antenna), C115 (match pad), R111 (0R RF series-match)
- Added J13 u.FL (Molex 73412-0110) + bias-tee: L8 27nH feed, C127 33pF DC block,
  C128 10nF VCC_RF bypass, D17 PESD0402-140 ESD (verify Vrwm >= 5 V)

Firmware:
- mdx_config.h: MDX_ITX_V_PER_A 0.4 -> 1.0 (INA241A2 is 50 V/V, not 20)
- hal_stm32.c: LSM6DSO32 accel init 0x48 -> 0x40 (FS_XL encoding differs; keeps +-4 g)
- make test: 96 checks pass

BOM: bom_data.json reconciled to the updated board (every placed part has an MPN;
fab BOM drops only the 15 test points). Regenerated JLCPCB fab package and the
DigiKey upload BOM (grouped by MPN, compact references).
Parts:
- removed C115: DNP (match, shunt), Capacitor_SMD:C_0402_1005Metric, symbol Device:C
- removed R111: 0R (match, series), Resistor_SMD:R_0402_1005Metric, symbol Device:R
- removed U28: GNSS chip antenna, RF_Antenna:Antenova_SR4G013_GPS, symbol Device:Antenna_Chip
- added C127: 33 pF, Capacitor_SMD:C_0402_1005Metric, symbol Device:C
- added C128: 10nF, Capacitor_SMD:C_0402_1005Metric, symbol Device:C
- added D17: PESD0402-140, Diode_SMD:D_0402_1005Metric, symbol Device:D_TVS
- added J13: Conn_Coaxial, Connector_Coaxial:U.FL_Molex_MCRF_73412-0110_Vertical, symbol Connector:Conn_Coaxial
- added L8: 27nH, Inductor_SMD:L_0402_1005Metric, symbol Device:L
- U23: value LSM6DSM (IMU) -> LSM6DSO32TR
Connections:
- net GND: now also C128.2, D17.1 (A1), J13.2 (Ext)
- net at U27.14 (VCC_RF): now also C128.1, L8.1
- net GNSS_RF: no longer names the net of U27.11 (RF_IN)
- net GNSS_RF: now also C127.1
- new net: C127.2, D17.2 (A2), J13.1 (In), L8.2
- no-connect marks 52 -> 51

Commit message: Add LL-audio + expansion-header support (firmware, schematic nets, mount holes)
Firmware (host bench 96/0):
- Optional low-latency audio module (nRF52840 daughterboard on J14): settings
  item "Low-latency audio" + "Pair LL headphones" (auto-exposed to UI and app via
  the item table), settings_t.ll_audio, HAL hal_ll_audio_*(), USART3 (PD8/PD9) +
  PG0/PG1 on the target; BM83 kept for BLE/app + standard-BT audio. Sim stubs.
- Expansion header: I2C4 (PF14/PF15), SPI2 (PB13/14/15, CS PG8), UART5 (PB6/PB12),
  GPIO PE13/PA15 initialised; portable hal_exp_*() API + sim stubs.

Schematic: J14 LL-audio header and expansion-header nets wired to the MCU; cleared
the no-connect flags on the newly used STM32 pins (PD8/9, PG0/1, PF14/15, PB13/14/15,
PG8, PB6, PB12, PE13, PA15).

Board: added 4x M3 (3.2 mm) mounting holes (H1-H4) to the main board at the
enclosure positions (128 x 85 mm rectangle, 3.55 mm inset).

Docs: firmware guide menu, design report (IMU), staged bring-up, and the priced BOM
review updated for the current part set.
Parts:
- added J14: BT LL Audio (optional), Connector_Samtec_MicroMate:Samtec_T1M-10-X-S-V_1x10-1MP_P1.0mm_Terminal_Vertical, symbol Connector_Generic:Conn_02x05_Odd_Even
- added J15: Expanson Header, Connector_Samtec_MicroMate:Samtec_T1M-12-X-S-V_1x12-1MP_P1.0mm_Terminal_Vertical, symbol Connector_Generic:Conn_02x06_Odd_Even
Connections:
- net +3V3: now also J14.1 (Pin_1), J15.1 (Pin_1)
- net GND: now also J14.10 (Pin_10), J14.2 (Pin_2), J15.2 (Pin_2)
- net I2S_BCLK: now also J14.3 (Pin_3)
- net I2S_DOUT: now also J14.5 (Pin_5)
- net I2S_LRCLK: now also J14.4 (Pin_4)
- new net EXP_GPIO1: J15.11 (Pin_11)
- new net EXP_GPIO2: J15.12 (Pin_12)
- new net EXP_I2C_SCL: J15.3 (Pin_3)
- new net EXP_I2C_SDA: J15.4 (Pin_4)
- new net EXP_SPI_CS: J15.8 (Pin_8)
- new net EXP_SPI_MISO: J15.7 (Pin_7)
- new net EXP_SPI_MOSI: J15.6 (Pin_6)
- new net EXP_SPI_SCK: J15.5 (Pin_5)
- new net EXP_UART_RX: J15.10 (Pin_10)
- new net EXP_UART_TX: J15.9 (Pin_9)
- new net NRF_RESET: J14.8 (Pin_8)
- new net NRF_RXD: J14.6 (Pin_6)
- new net NRF_STATUS: J14.9 (Pin_9)
- new net NRF_TXD: J14.7 (Pin_7)
